File: wafflehw_rev0.1/wafflehw_rev0.1.kicad_pcb (KiCad board)
At the start: 2 copper layers, 42 x 66 mm, 41 parts, among them J2 OLED_Disp, J3 FH34SRJ-30S-0.5SH, J4 BATT, J5 LCD_BL, Q1 AO3400A, Q2 AO3400A, Q3 AO3400A, SW1 SW_Push, SW2 BTN_UP, SW3 BTN_DN, SW4 BTN_OK, U1 Ai-Thinker-Ra-01, U2 TP4054, U3 ESP32-S3-WROOM-1, U4 MD57E33QA3, U5 MD57E33QA3

Commit message: Routed v 0.1
Parts:
- added M1: Motor_DC, Jumper:SolderJumper-2_P1.3mm_Open_RoundedPad1.0x1.5mm, F.Cu at (133.8, 38.5)
- moved C3 47.5 mm to (106.5, 84.0)
- moved Q3 10.4 mm to (132.5, 55.0)
- moved BUZZER1 0.81 mm to (121.1, 38.1), turned to 0 degrees
Routing:
- net GND: track 34.2 -> 246.7 mm, vias 10 -> 54
- net +3.3V: track 21.0 -> 95.8 mm, vias 2 -> 4
- net RADIO_DIO0: track 0.00 -> 71.5 mm, vias 0 -> 2
- net ESP32_D-: track 0.00 -> 61.9 mm, vias 0 -> 2
- net ESP32_D+: track 0.57 -> 58.7 mm, vias 1 -> 2
- net RADIO_RST: track 0.00 -> 58.0 mm, vias 0 -> 2
- net VBAT_STATUS: track 0.00 -> 54.1 mm, vias 0 -> 2
- net +BATT: track 51.8 -> 105.7 mm, vias 0 -> 2
- net BTN_DOWN: track 0.00 -> 48.8 mm, vias 0 -> 3
- net BTN_UP: track 0.00 -> 47.3 mm, vias 0 -> 1
- net RADIO_DIO2: track 0.00 -> 47.1 mm, vias 0 -> 2
- net RADIO_DIO1: track 0.00 -> 45.5 mm, vias 0 -> 2
- net LCD_LED: track 0.00 -> 41.6 mm, vias 0 -> 2
- net VIBRATE: track 0.00 -> 38.8 mm, vias 0 -> 2
- net BTN_OK: track 0.00 -> 36.9 mm, vias 0 -> 1
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