File: wafflehw_rev0.1/wafflehw_rev0.1.kicad_sch (KiCad schematic)
At the start: 42 parts, among them J2 OLED_Disp, J3 FH34SRJ-30S-0.5SH, J4 BATT, J5 LCD_BL, M1 Motor_DC, Q1 AO3400A, Q2 AO3400A, Q3 AO3400A, SW1 SW_Push, SW2 BTN_UP, SW3 BTN_DN, SW4 BTN_OK, U1 Ai-Thinker-Ra-01, U2 TP4054, U3 ESP32-S3-WROOM-1, U4 MD57E33QA3, U5 MD57E33QA3

Commit message: Routed v 0.1
Parts:
- M1: footprint (none) -> Jumper:SolderJumper-2_P1.3mm_Open_RoundedPad1.0x1.5mm
Changed lines of the file:
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@@
 		)
 		(instances
-			(project ""
+			(project "wafflehw_rev0.1"
 				(path "/4ff13b59-a364-4b9f-8d1b-d43f091608d9"
 					(reference "U4")
@@
 		)
 		(instances
-			(project ""
+			(project "wafflehw_rev0.1"
 				(path "/4ff13b59-a364-4b9f-8d1b-d43f091608d9"
 					(reference "C7")
@@
 		)
 		(instances
-			(project ""
+			(project "wafflehw_rev0.1"
 				(path "/4ff13b59-a364-4b9f-8d1b-d43f091608d9"
 					(reference "#PWR016")
@@
 		)
 		(instances
-			(project ""
+			(project "wafflehw_rev0.1"
 				(path "/4ff13b59-a364-4b9f-8d1b-d43f091608d9"
 					(reference "#PWR015")
@@
 		)
 		(instances
-			(project ""
+			(project "wafflehw_rev0.1"
 				(path "/4ff13b59-a364-4b9f-8d1b-d43f091608d9"
 					(reference "#PWR020")
@@
 		)
 		(instances
-			(project ""
+			(project "wafflehw_rev0.1"
 				(path "/4ff13b59-a364-4b9f-8d1b-d43f091608d9"
 					(reference "#PWR018")
@@
 		)
 		(instances
-			(project ""
+			(project "wafflehw_rev0.1"
 				(path "/4ff13b59-a364-4b9f-8d1b-d43f091608d9"
 					(reference "#PWR08")
@@
 		)
 		(instances
-			(project ""
+			(project "wafflehw_rev0.1"
 				(path "/4ff13b59-a364-4b9f-8d1b-d43f091608d9"
 					(reference "#PWR013")
@@
 		)
 		(instances
-			(project ""
+			(project "wafflehw_rev0.1"
 				(path "/4ff13b59-a364-4b9f-8d1b-d43f091608d9"
 					(reference "C3")
@@
 		)
 		(instances
-			(project ""
+			(project "wafflehw_rev0.1"
 				(path "/4ff13b59-a364-4b9f-8d1b-d43f091608d9"
 					(reference "U2")
@@
 		)
 		(instances
-			(project ""
+			(project "wafflehw_rev0.1"
 				(path "/4ff13b59-a364-4b9f-8d1b-d43f091608d9"
 					(reference "U3")
@@
 		)
 		(instances
-			(project ""
+			(project "wafflehw_rev0.1"
 				(path "/4ff13b59-a364-4b9f-8d1b-d43f091608d9"
 					(reference "#PWR028")
@@
 		)
 		(instances
-			(project ""
+			(project "wafflehw_rev0.1"
 				(path "/4ff13b59-a364-4b9f-8d1b-d43f091608d9"
 					(reference "Q1")
@@
 		)
 		(instances
-			(project ""
+			(project "wafflehw_rev0.1"
 				(path "/4ff13b59-a364-4b9f-8d1b-d43f091608d9"
 					(reference "J5")
@@
 		)
 		(instances
-			(project ""
+			(project "wafflehw_rev0.1"
 				(path "/4ff13b59-a364-4b9f-8d1b-d43f091608d9"
 					(reference "R2")
@@
 		)
 		(instances
-			(project ""
+			(project "wafflehw_rev0.1"
 				(path "/4ff13b59-a364-4b9f-8d1b-d43f091608d9"
 					(reference "#PWR01")
@@
 		)
 		(instances
-			(project ""
+			(project "wafflehw_rev0.1"
 				(path "/4ff13b59-a364-4b9f-8d1b-d43f091608d9"
 					(reference "C6")
@@
 		)
 		(instances
-			(project ""
+			(project "wafflehw_rev0.1"
 				(path "/4ff13b59-a364-4b9f-8d1b-d43f091608d9"
 					(reference "C10")
@@
 		)
 		(instances
-			(project ""
+			(project "wafflehw_rev0.1"
 				(path "/4ff13b59-a364-4b9f-8d1b-d43f091608d9"
 					(reference "#PWR026")
@@
 		)
 		(instances
-			(project ""
+			(project "wafflehw_rev0.1"
 				(path "/4ff13b59-a364-4b9f-8d1b-d43f091608d9"
 					(reference "J2")
@@
 		)
 		(instances
-			(project ""
+			(project "wafflehw_rev0.1"
 				(path "/4ff13b59-a364-4b9f-8d1b-d43f091608d9"
 					(reference "USB1")
@@
 		)
 		(instances
-			(project ""
+			(project "wafflehw_rev0.1"
 				(path "/4ff13b59-a364-4b9f-8d1b-d43f091608d9"
 					(reference "#PWR04")
@@
 		)
 		(instances
-			(project ""
+			(project "wafflehw_rev0.1"
 				(path "/4ff13b59-a364-4b9f-8d1b-d43f091608d9"
 					(reference "R4")
@@
 		)
 		(instances
-			(project ""
+			(project "wafflehw_rev0.1"
 				(path "/4ff13b59-a364-4b9f-8d1b-d43f091608d9"
 					(reference "#PWR024")
@@
 		)
 		(instances
-			(project "Waffle2Rev0.1"
+			(project "wafflehw_rev0.1"
 				(path "/4ff13b59-a364-4b9f-8d1b-d43f091608d9"
 					(reference "#PWR09")
@@
 		)
 		(instances
-			(project ""
+			(project "wafflehw_rev0.1"
 				(path "/4ff13b59-a364-4b9f-8d1b-d43f091608d9"
 					(reference "J3")
@@
 		)
 		(instances
-			(project ""
+			(project "wafflehw_rev0.1"
 				(path "/4ff13b59-a364-4b9f-8d1b-d43f091608d9"
 					(reference "#PWR07")
@@
 		)
 		(instances
-			(project ""
+			(project "wafflehw_rev0.1"
 				(path "/4ff13b59-a364-4b9f-8d1b-d43f091608d9"
 					(reference "SW4")
@@
 		)
 		(instances
-			(project ""
+			(project "wafflehw_rev0.1"
 				(path "/4ff13b59-a364-4b9f-8d1b-d43f091608d9"
 					(reference "#PWR03")
@@
 		)
 		(instances
-			(project ""
+			(project "wafflehw_rev0.1"
 				(path "/4ff13b59-a364-4b9f-8d1b-d43f091608d9"
 					(reference "#PWR011")
@@
 		)
 		(instances
-			(project ""
+			(project "wafflehw_rev0.1"
 				(path "/4ff13b59-a364-4b9f-8d1b-d43f091608d9"
 					(reference "C12")
@@
 		)
 		(instances
-			(project ""
+			(project "wafflehw_rev0.1"
 				(path "/4ff13b59-a364-4b9f-8d1b-d43f091608d9"
 					(reference "D1")
@@
 		)
 		(instances
-			(project ""
+			(project "wafflehw_rev0.1"
 				(path "/4ff13b59-a364-4b9f-8d1b-d43f091608d9"
 					(reference "#PWR05")
@@
 		)
 		(instances
-			(project ""
+			(project "wafflehw_rev0.1"
 				(path "/4ff13b59-a364-4b9f-8d1b-d43f091608d9"
 					(reference "SW3")
@@
 		)
 		(instances
-			(project ""
+			(project "wafflehw_rev0.1"
 				(path "/4ff13b59-a364-4b9f-8d1b-d43f091608d9"
 					(reference "#PWR017")
@@
 		)
 		(instances
-			(project ""
+			(project "wafflehw_rev0.1"
 				(path "/4ff13b59-a364-4b9f-8d1b-d43f091608d9"
 					(reference "#PWR029")
@@
 		)
 		(instances
-			(project ""
+			(project "wafflehw_rev0.1"
 				(path "/4ff13b59-a364-4b9f-8d1b-d43f091608d9"
 					(reference "#PWR014")
@@
 		)
 		(instances
-			(project ""
+			(project "wafflehw_rev0.1"
 				(path "/4ff13b59-a364-4b9f-8d1b-d43f091608d9"
 					(reference "R3")
@@
 		)
 		(instances
-			(project ""
+			(project "wafflehw_rev0.1"
 				(path "/4ff13b59-a364-4b9f-8d1b-d43f091608d9"
 					(reference "SW1")
@@
 		)
 		(instances
-			(project ""
+			(project "wafflehw_rev0.1"
 				(path "/4ff13b59-a364-4b9f-8d1b-d43f091608d9"
 					(reference "C1")
@@
 		)
 		(instances
-			(project ""
+			(project "wafflehw_rev0.1"
 				(path "/4ff13b59-a364-4b9f-8d1b-d43f091608d9"
 					(reference "#PWR025")
@@
 		)
 		(instances
-			(project ""
+			(project "wafflehw_rev0.1"
 				(path "/4ff13b59-a364-4b9f-8d1b-d43f091608d9"
 					(reference "SW2")
@@
 		)
 		(instances
-			(project ""
+			(project "wafflehw_rev0.1"
 				(path "/4ff13b59-a364-4b9f-8d1b-d43f091608d9"
 					(reference "#PWR033")
@@
 		)
 		(instances
-			(project ""
+			(project "wafflehw_rev0.1"
 				(path "/4ff13b59-a364-4b9f-8d1b-d43f091608d9"
 					(reference "D2")
@@
 		)
 		(instances
-			(project ""
+			(project "wafflehw_rev0.1"
 				(path "/4ff13b59-a364-4b9f-8d1b-d43f091608d9"
 					(reference "J4")
@@
 		)
 		(instances
-			(project ""
+			(project "wafflehw_rev0.1"
 				(path "/4ff13b59-a364-4b9f-8d1b-d43f091608d9"
 					(reference "#PWR022")
@@
 		)
 		(instances
-			(project ""
+			(project "wafflehw_rev0.1"
 				(path "/4ff13b59-a364-4b9f-8d1b-d43f091608d9"
 					(reference "#PWR06")
@@
 		)
 		(instances
-			(project ""
+			(project "wafflehw_rev0.1"
 				(path "/4ff13b59-a364-4b9f-8d1b-d43f091608d9"
 					(reference "C2")
@@
 		)
 		(instances
-			(project ""
+			(project "wafflehw_rev0.1"
 				(path "/4ff13b59-a364-4b9f-8d1b-d43f091608d9"
 					(reference "AE1")
@@
 		)
 		(instances
-			(project "Waffle2Rev0.1"
+			(project "wafflehw_rev0.1"
 				(path "/4ff13b59-a364-4b9f-8d1b-d43f091608d9"
 					(reference "#PWR023")
@@
 		)
 		(instances
-			(project ""
+			(project "wafflehw_rev0.1"
 				(path "/4ff13b59-a364-4b9f-8d1b-d43f091608d9"
 					(reference "C8")
@@
 		)
 		(instances
-			(project ""
+			(project "wafflehw_rev0.1"
 				(path "/4ff13b59-a364-4b9f-8d1b-d43f091608d9"
 					(reference "C4")
@@
 		)
 		(instances
-			(project ""
+			(project "wafflehw_rev0.1"
 				(path "/4ff13b59-a364-4b9f-8d1b-d43f091608d9"
 					(reference "#PWR019")
@@
 		)
 		(instances
-			(project ""
+			(project "wafflehw_rev0.1"
 				(path "/4ff13b59-a364-4b9f-8d1b-d43f091608d9"
 					(reference "FB1")
@@
 		)
 		(instances
-			(project ""
+			(project "wafflehw_rev0.1"
 				(path "/4ff13b59-a364-4b9f-8d1b-d43f091608d9"
 					(reference "C5")
@@
 		)
 		(instances
-			(project "Waffle2Rev0.1"
+			(project "wafflehw_rev0.1"
 				(path "/4ff13b59-a364-4b9f-8d1b-d43f091608d9"
 					(reference "#PWR010")
@@
 			)
 		)
-		(property "Footprint" ""
+		(property "Footprint" "Jumper:SolderJumper-2_P1.3mm_Open_RoundedPad1.0x1.5mm"
 			(at 39.37 101.346 0)
 			(effects
@@
 		)
 		(instances
-			(project ""
+			(project "wafflehw_rev0.1"
 				(path "/4ff13b59-a364-4b9f-8d1b-d43f091608d9"
 					(reference "M1")
@@
 		)
 		(instances
-			(project ""
+			(project "wafflehw_rev0.1"
 				(path "/4ff13b59-a364-4b9f-8d1b-d43f091608d9"
 					(reference "#PWR02")
@@
 		)
 		(instances
-			(project ""
+			(project "wafflehw_rev0.1"
 				(path "/4ff13b59-a364-4b9f-8d1b-d43f091608d9"
 					(reference "R1")
@@
 		)
 		(instances
-			(project ""
+			(project "wafflehw_rev0.1"
 				(path "/4ff13b59-a364-4b9f-8d1b-d43f091608d9"
 					(reference "#PWR027")
@@
 		)
 		(instances
-			(project ""
+			(project "wafflehw_rev0.1"
 				(path "/4ff13b59-a364-4b9f-8d1b-d43f091608d9"
 					(reference "U1")
@@
 		)
 		(instances
-			(project ""
+			(project "wafflehw_rev0.1"
 				(path "/4ff13b59-a364-4b9f-8d1b-d43f091608d9"
 					(reference "BUZZER1")
@@
 		)
 		(instances
-			(project ""
+			(project "wafflehw_rev0.1"
 				(path "/4ff13b59-a364-4b9f-8d1b-d43f091608d9"
 					(reference "#PWR030")
@@
 		)
 		(instances
-			(project ""
+			(project "wafflehw_rev0.1"
 				(path "/4ff13b59-a364-4b9f-8d1b-d43f091608d9"
 					(reference "#PWR021")
